Commit message: Corrected toro urdf model and retuned model

File: resources/toro/toro.urdf (robot description, URDF)
Before this commit: robot DLR_TORO, 34 links, 33 joints
Joints:
- joint j12: origin xyz=-0.0000000000 0.0000000000 -0.1189000000 rpy=0 0 0 -> xyz=-0.0000000000 0.0000000000 -0.0200000 rpy=0 0 0
- joint j27: origin xyz=0.056 0 0.1877 -> xyz=-0.035 0 0.05
- joint j6: origin xyz=-0.0000000000 -0.0000000000 -0.1189000000 rpy=0 0 0 -> xyz=-0.0000000000 0.0000000000 -0.0200000 rpy=0 0 0

Commit message: Updated toro head weight

File: resources/toro/toro.urdf (robot description, URDF)
Before this commit: robot DLR_TORO, 34 links, 33 joints
Links:
- link neck_link2: mass 1.4522900000 -> 2.4522900000
